File: schematics/rc_rx_3_3V_with_gyro_iface_and_rear_H-bridge.sch (EAGLE design)
At the start: 45 parts, among them IC1 PIC16F1826/27SO, IC2 LD117AS50TR, Q1 IRF3704S, Q2 IRF3704S, Q3 IRF7309, Q4 IRF7309, Q5 BSS123, Q6 BSS123

Commit message: Working on broken ADC and MSSP
This commit is to show to Microchip
Parts:
- removed Q5, Q6: BSS123, transistor-small-signal:BSS123
- removed R21, R22, R23, R24: 4k7, resistor:R-EU_M0805
- added C3: 4.7uF, rcl:CPOL-EUE1.8-4
- added C4: 100nF, rcl:C-USC0805
- added C5, C6: 0.1uF, rcl:C-EUC0805
- added IC3: 78L05F, linear:78L05F
- C1: device rcl:C-US025-025X050 -> rcl:C-USC0805
- R14, R15: value 1k -> 470
Connections:
- new net +12V: C6.1, IC3.VI
- net 3.3V: now also C3.+, C5.1, IC3.VO; no longer Q5.G, Q6.G, R21.1, R22.1
- net 5V: now also C4.1; no longer C2.+
- net GND: now also C3.-, C4.2, C5.2, C6.2, IC3.GND, IC3.GND@1
- net SCL_3.3: no longer Q6.S, R22.2
- net SCL_5: no longer Q6.D, R24.2
- net SDA_3.3: no longer Q5.S, R21.2
- net SDA_5: no longer Q5.D, R23.2
- net V+: now also C2.+
- net VDD: no longer R23.1, R24.1
Other:
- moved on the sheet: C1, C2
