File: schematics/rc_rx_5V_rotors_only.brd (EAGLE design)
At the start: 100 x 80 mm, 28 parts, among them IC1 PIC16F1826/27P, IC2 LD117AS50TR, Q1 IRF3704S, Q2 IRF3704S

Commit message: Working on broken ADC and MSSP
This commit is to show to Microchip
Connections:
- removed net PGC: IC1.12, JP4.1
- removed net PGD: IC1.13, JP4.2
- new net LED: IC1.17
- new net SCL1: IC1.10
- new net SDA1: IC1.7
- net CH1_IN: now also IC1.12, JP4.1; no longer IC1.7
- net CH3_IN: now also IC1.13, JP4.2; no longer IC1.10
Changed lines of the file:
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@@
 <signals>
 <signal name="CH3_IN">
-<contactref element="IC1" pad="10"/>
 <contactref element="R11" pad="2"/>
-<wire x1="41.91" y1="40.64" x2="41.91" y2="43.18" width="0" layer="19" extent="1-1"/>
+<contactref element="IC1" pad="13"/>
+<contactref element="JP4" pad="2"/>
+<wire x1="34.29" y1="40.64" x2="41.91" y2="43.18" width="0" layer="19" extent="1-1"/>
+<wire x1="39.37" y1="22.86" x2="34.29" y2="40.64" width="0" layer="19" extent="1-1"/>
 </signal>
 <signal name="GND">
@@
 <wire x1="10.16" y1="36.83" x2="10.16" y2="26.67" width="0" layer="19" extent="1-1"/>
 </signal>
-<signal name="PGD">
-<contactref element="JP4" pad="2"/>
-<contactref element="IC1" pad="13"/>
-<wire x1="39.37" y1="22.86" x2="34.29" y2="40.64" width="0" layer="19" extent="1-1"/>
-</signal>
-<signal name="PGC">
+<signal name="CH1_IN">
+<contactref element="R9" pad="2"/>
+<contactref element="IC1" pad="12"/>
 <contactref element="JP4" pad="1"/>
-<contactref element="IC1" pad="12"/>
-<wire x1="41.91" y1="22.86" x2="36.83" y2="40.64" width="0" layer="19" extent="1-1"/>
-</signal>
-<signal name="CH1_IN">
-<contactref element="IC1" pad="7"/>
-<contactref element="R9" pad="2"/>
-<wire x1="36.83" y1="26.67" x2="36.83" y2="33.02" width="0" layer="19" extent="1-1"/>
+<wire x1="36.83" y1="26.67" x2="36.83" y2="40.64" width="0" layer="19" extent="1-1"/>
+<wire x1="41.91" y1="22.86" x2="36.83" y2="26.67" width="0" layer="19" extent="1-1"/>
 </signal>
 <signal name="CH2_IN">
@@
 <wire x1="24.13" y1="22.86" x2="41.91" y2="50.8" width="0" layer="19" extent="1-1"/>
 </signal>
+<signal name="LED">
+<contactref element="IC1" pad="17"/>
+</signal>
+<signal name="SDA1">
+<contactref element="IC1" pad="7"/>
+</signal>
+<signal name="SCL1">
+<contactref element="IC1" pad="10"/>
+</signal>
 </signals>
